Commit message: Updated for ROS 2 Humble Support

File: tortoisebot_description/models/urdf/tortoisebot.xacro (robot description, xacro)
@@ -14,5 +14,5 @@
 			<origin rpy="0 0 0" xyz="0 0 0"/>
 			<geometry>
-				<mesh filename="file://$(find tortoisebot_description)/meshes/base_link.stl" scale="0.001 0.001 0.001"/>
+				<mesh filename="file://$(find tortoisebot_description)/models/meshes/base_link.stl" scale="0.001 0.001 0.001"/>
 			</geometry>
 			<material name="grey"/>
@@ -21,5 +21,5 @@
 			<origin rpy="0 0 0" xyz="0 0 0"/>
 			<geometry>
-				<mesh filename="file://$(find tortoisebot_description)/meshes/base_link.stl" scale="0.001 0.001 0.001"/>
+				<mesh filename="file://$(find tortoisebot_description)/models/meshes/base_link.stl" scale="0.001 0.001 0.001"/>
 			</geometry>
 		</collision>
@@ -34,5 +34,5 @@
 			<origin rpy="0 0 0" xyz="-0.0325 0.07073 -0.03245"/>
 			<geometry>
-				<mesh filename="file://$(find tortoisebot_description)/meshes/wheel_right.stl" scale="0.001 0.001 0.001"/>
+				<mesh filename="file://$(find tortoisebot_description)/models/meshes/wheel_right.stl" scale="0.001 0.001 0.001"/>
 			</geometry>
 			<material name="black"/>
@@ -41,5 +41,5 @@
 			<origin rpy="0 0 0" xyz="-0.0325 0.07073 -0.03245"/>
 			<geometry>
-				<mesh filename="file://$(find tortoisebot_description)/meshes/wheel_right.stl" scale="0.001 0.001 0.001"/>
+				<mesh filename="file://$(find tortoisebot_description)/models/meshes/wheel_right.stl" scale="0.001 0.001 0.001"/>
 			</geometry>
 		</collision>
@@ -54,5 +54,5 @@
 			<origin rpy="0 0 0" xyz="-0.0325 -0.07073 -0.03245"/>
 			<geometry>
-				<mesh filename="file://$(find tortoisebot_description)/meshes/wheel_left.stl" scale="0.001 0.001 0.001"/>
+				<mesh filename="file://$(find tortoisebot_description)/models/meshes/wheel_left.stl" scale="0.001 0.001 0.001"/>
 			</geometry>
 			<material name="black"/>
@@ -61,5 +61,5 @@
 			<origin rpy="0 0 0" xyz="-0.0325 -0.07073 -0.03245"/>
 			<geometry>
-				<mesh filename="file://$(find tortoisebot_description)/meshes/wheel_left.stl" scale="0.001 0.001 0.001"/>
+				<mesh filename="file://$(find tortoisebot_description)/models/meshes/wheel_left.stl" scale="0.001 0.001 0.001"/>
 			</geometry>
 		</collision>
@@ -74,5 +74,5 @@
 			<origin rpy="0 0 0" xyz="0.032 -0.0 -0.01915"/>
 			<geometry>
-				<mesh filename="file://$(find tortoisebot_description)/meshes/caster.stl" scale="0.001 0.001 0.001"/>
+				<mesh filename="file://$(find tortoisebot_description)/models/meshes/caster.stl" scale="0.001 0.001 0.001"/>
 			</geometry>
 			<material name="black"/>
@@ -81,5 +81,5 @@
 			<origin rpy="0 0 0" xyz="0.032 -0.0 -0.01915"/>
 			<geometry>
-				<mesh filename="file://$(find tortoisebot_description)/meshes/caster.stl" scale="0.001 0.001 0.001"/>
+				<mesh filename="file://$(find tortoisebot_description)/models/meshes/caster.stl" scale="0.001 0.001 0.001"/>
 			</geometry>
 		</collision>
@@ -94,5 +94,5 @@
 			<origin rpy="0 0 0" xyz="0.022 -0.031 -0.14715"/>
 			<geometry>
-				<mesh filename="file://$(find tortoisebot_description)/meshes/lidar_body.stl" scale="0.001 0.001 0.001"/>
+				<mesh filename="file://$(find tortoisebot_description)/models/meshes/lidar_body.stl" scale="0.001 0.001 0.001"/>
 			</geometry>
 			<material name="black"/>
@@ -101,5 +101,5 @@
 			<origin rpy="0 0 0" xyz="0.022 -0.031 -0.14715"/>
 			<geometry>
-				<mesh filename="file://$(find tortoisebot_description)/meshes/lidar_body.stl" scale="0.001 0.001 0.001"/>
+				<mesh filename="file://$(find tortoisebot_description)/models/meshes/lidar_body.stl" scale="0.001 0.001 0.001"/>
 			</geometry>
 		</collision>
@@ -114,5 +114,5 @@
 			<origin rpy="0 0 0" xyz="-0.05 -0.0 -0.18065"/>
 			<geometry>
-				<mesh filename="file://$(find tortoisebot_description)/meshes/lidar_motorend.stl" scale="0.001 0.001 0.001"/>
+				<mesh filename="file://$(find tortoisebot_description)/models/meshes/lidar_motorend.stl" scale="0.001 0.001 0.001"/>
 			</geometry>
 			<material name="blue"/>
@@ -121,5 +121,5 @@
 			<origin rpy="0 0 0" xyz="-0.05 -0.0 -0.18065"/>
 			<geometry>
-				<mesh filename="file://$(find tortoisebot_description)/meshes/lidar_motorend.stl" scale="0.001 0.001 0.001"/>
+				<mesh filename="file://$(find tortoisebot_description)/models/meshes/lidar_motorend.stl" scale="0.001 0.001 0.001"/>
 			</geometry>
 		</collision>
@@ -134,5 +134,5 @@
 			<origin rpy="0 0 0" xyz="0.0 -0.0 -0.18065"/>
 			<geometry>
-				<mesh filename="file://$(find tortoisebot_description)/meshes/lidar_bottom.stl" scale="0.001 0.001 0.001"/>
+				<mesh filename="file://$(find tortoisebot_description)/models/meshes/lidar_bottom.stl" scale="0.001 0.001 0.001"/>
 			</geometry>
 			<material name="blue"/>
@@ -141,5 +141,5 @@
 			<origin rpy="0 0 0" xyz="0.0 -0.0 -0.18065"/>
 			<geometry>
-				<mesh filename="file://$(find tortoisebot_description)/meshes/lidar_bottom.stl" scale="0.001 0.001 0.001"/>
+				<mesh filename="file://$(find tortoisebot_description)/models/meshes/lidar_bottom.stl" scale="0.001 0.001 0.001"/>
 			</geometry>
 		</collision>
@@ -154,5 +154,5 @@
 			<origin rpy="0 0 0" xyz="0.0 -0.0 -0.19615"/>
 			<geometry>
-				<mesh filename="file://$(find tortoisebot_description)/meshes/lidar_top.stl" scale="0.001 0.001 0.001"/>
+				<mesh filename="file://$(find tortoisebot_description)/models/meshes/lidar_top.stl" scale="0.001 0.001 0.001"/>
 			</geometry>
 			<material name="blue"/>
@@ -161,5 +161,5 @@
 			<origin rpy="0 0 0" xyz="0.0 -0.0 -0.19615"/>
 			<geometry>
-				<mesh filename="file://$(find tortoisebot_description)/meshes/lidar_top.stl" scale="0.001 0.001 0.001"/>
+				<mesh filename="file://$(find tortoisebot_description)/models/meshes/lidar_top.stl" scale="0.001 0.001 0.001"/>
 			</geometry>
 		</collision>
@@ -174,5 +174,5 @@
 			<origin rpy="0 0 0" xyz="-0.04 0.01025 -0.10543"/>
 			<geometry>
-				<mesh filename="file://$(find tortoisebot_description)/meshes/imu.stl" scale="0.001 0.001 0.001"/>
+				<mesh filename="file://$(find tortoisebot_description)/models/meshes/imu.stl" scale="0.001 0.001 0.001"/>
 			</geometry>
 			<material name="grey"/>
@@ -181,5 +181,5 @@
 			<origin rpy="0 0 0" xyz="-0.04 0.01025 -0.10543"/>
 			<geometry>
-				<mesh filename="file://$(find tortoisebot_description)/meshes/imu.stl" scale="0.001 0.001 0.001"/>
+				<mesh filename="file://$(find tortoisebot_description)/models/meshes/imu.stl" scale="0.001 0.001 0.001"/>
 			</geometry>
 		</collision>
@@ -194,5 +194,5 @@
 			<origin rpy="0 0 0" xyz="-0.061 -0.0 -0.11515"/>
 			<geometry>
-				<mesh filename="file://$(find tortoisebot_description)/meshes/camera.stl" scale="0.001 0.001 0.001"/>
+				<mesh filename="file://$(find tortoisebot_description)/models/meshes/camera.stl" scale="0.001 0.001 0.001"/>
 			</geometry>
 			<material name="grey"/>
@@ -201,5 +201,5 @@
 			<origin rpy="0 0 0" xyz="-0.061 -0.0 -0.11515"/>
 			<geometry>
-				<mesh filename="file://$(find tortoisebot_description)/meshes/camera.stl" scale="0.001 0.001 0.001"/>
+				<mesh filename="file://$(find tortoisebot_description)/models/meshes/camera.stl" scale="0.001 0.001 0.001"/>
 			</geometry>
 		</collision>
